Commit message: Changed urdf to take yaml params

File: nuturtle_description/urdf/turtlebot3_burger.urdf.xacro (robot description, xacro)
@@ -2,4 +2,14 @@
 <robot xmlns:xacro="http://ros.org/wiki/xacro" name="turtlebot3_burger">
   <!-- <xacro:include filename="$(find turtlebot3_description)/urdf/common_properties.urdf"/> -->
+<xacro:property name="yaml_file" value="$(find nuturtle_description)/config/diff_params.yaml" />
+<xacro:property name="props" value="${xacro.load_yaml(yaml_file)}" />
+<xacro:property name="start"  value="${props['/**']}" />
+<xacro:property name="ros__parameters"  value="${start['ros__parameters']}" />
+<xacro:property name="wheelradius"  value="${ros__parameters['wheelradius']}" />
+<xacro:property name="track_width"  value="${ros__parameters['track_width']}" />
+<xacro:property name="motor_cmd_max"  value="${ros__parameters['motor_cmd_max']}" />
+<xacro:property name="motor_cmd_per_rad_sec"  value="${ros__parameters['motor_cmd_per_rad_sec']}" />
+<xacro:property name="encoder_ticks_per_rad"  value="${ros__parameters['encoder_ticks_per_rad']}" />
+<xacro:property name="collision_radius"  value="${ros__parameters['collision_radius']}" />
   <!-- Init colour -->
   <material name="black">
@@ -50,5 +60,10 @@
       <origin xyz="-0.032 0 0.070" rpy="0 0 0"/>
       <geometry>
-        <box size="0.140 0.140 0.143"/>
+        <xacro:if value = "${collision_radius &gt; 0.0}">
+          <cylinder length="0.143" radius="${collision_radius}"/>
+        </xacro:if>
+        <xacro:if value = "${collision_radius &lt; 0.0}">
+          <box size="0.140 0.140 0.143"/>
+        </xacro:if>
       </geometry>
     </collision>
@@ -62,5 +77,5 @@
     <parent link="base_link"/>
     <child link="wheel_left_link"/>
-    <origin xyz="0.0 0.08 0.023" rpy="-1.57 0 0"/>
+    <origin xyz="0.0 ${track_width/2} 0.023" rpy="-1.57 0 0"/>
     <axis xyz="0 0 1"/>
   </joint>
@@ -76,5 +91,5 @@
       <origin xyz="0 0 0" rpy="0 0 0"/>
       <geometry>
-        <cylinder length="0.018" radius="0.033"/>
+        <cylinder length="0.018" radius="${wheelradius}"/>
       </geometry>
     </collision>
@@ -88,5 +103,5 @@
     <parent link="base_link"/>
     <child link="wheel_right_link"/>
-    <origin xyz="0.0 -0.080 0.023" rpy="-1.57 0 0"/>
+    <origin xyz="0.0 -${track_width/2} 0.023" rpy="-1.57 0 0"/>
     <axis xyz="0 0 1"/>
   </joint>
@@ -102,5 +117,5 @@
       <origin xyz="0 0 0" rpy="0 0 0"/>
       <geometry>
-        <cylinder length="0.018" radius="0.033"/>
+        <cylinder length="0.018" radius="${wheelradius}"/>
       </geometry>
     </collision>

Commit message: Cant get arggument pipeline between launch file and xacro

File: nuturtle_description/urdf/turtlebot3_burger.urdf.xacro (robot description, xacro)
@@ -12,4 +12,5 @@
 <xacro:property name="encoder_ticks_per_rad"  value="${ros__parameters['encoder_ticks_per_rad']}" />
 <xacro:property name="collision_radius"  value="${ros__parameters['collision_radius']}" />
+<xacro:arg name="color" default="orange"/>
   <!-- Init colour -->
   <material name="black">
@@ -43,4 +44,7 @@
     <color rgba="1.0 1.0 1.0 1.0"/>
   </material>
+  <material name="purple">
+    <color rgba="0.3 0.16 0.52 1.0"/>
+  </material>
   <link name="base_footprint"/>
   <joint name="base_joint" type="fixed">
@@ -55,5 +59,5 @@
         <mesh filename="package://nuturtle_description/meshes/burger_base.stl" scale="0.001 0.001 0.001"/>
       </geometry>
-      <material name="light_black"/>
+      <material name="$(arg color)"/>
     </visual>
     <collision>
